Commit message: Fix Launch Warnings

File: hector_quadrotor_description/urdf/quadrotor_base.urdf.xacro (robot description, xacro)
@@ -5,4 +5,5 @@
   <!-- Main quadrotor link -->
   <xacro:macro name="quadrotor_base_macro">
+    <link name="dummy"/>
     <link name="base_link">
       <inertial>
@@ -24,4 +25,8 @@
       </collision>
     </link>
+    <joint name="dummy_joint" type="fixed">
+      <parent link="dummy"/>
+      <child link="base_link"/>
+    </joint>
     <!-- Sonar height sensor -->
     <xacro:sonar_sensor name="sonar" parent="base_link" ros_topic="sonar_height" update_rate="10" min_range="0.03" max_range="3.0" field_of_view="${40*pi/180}" ray_count="3">
